File: Circuito-IO/DomPiWeb.kicad_pcb (KiCad board)
At the start: 2 copper layers, 90 x 55 mm, 84 parts, among them J1 12V in, J10 Bx3, J11 Bx2, J12 Bx3, J2 5V out, J3 CONUFL001-SMD-T (Linx), J4 5v switch, J5 SIM7050, J6 RaspberryPi GPIO, J7 SIMDBG, J8 EXP1, J9 Bx2, Q1 DMG2305UXQ6, Q2 DMG2305UXQ6, U1 LM2596S-ADJ, U2 SIM900

Commit message: Correcciones del prototipo
Correcciones del prototipo
Parts:
- J1: value 12V in -> Entrada 12v
- J2: value 5V out -> Salida 5v
- J4: value 5v switch -> Salida 5v Controlada
- R10, R11, R12: value 22 -> 33
- moved R4 5.34 mm to (146.6, 70.5), turned to 270 degrees
- moved D1 4.15 mm to (143.7, 71.5), turned to 90 degrees
- moved Q2 3.91 mm to (116.0, 80.7), turned to 0 degrees
- moved R17 3.86 mm to (111.8, 80.7), turned to 270 degrees
- moved Q1 2.07 mm to (151.2, 70.5), turned to 0 degrees
- moved J8 2.00 mm to (137.0, 69.0)
- moved C8 1.76 mm to (139.2, 70.3)
Connections:
- Q1 pad 2: Net-(C1-Pad2) -> Net-(D1-Pad1)
- Q1 pad 3: Net-(D1-Pad1) -> Net-(C1-Pad2)
- Q2 pad 2: Net-(C6-Pad1) -> +5VD
- Q2 pad 3: +5VD -> Net-(C6-Pad1)
Routing:
- net Net-(D7-Pad1): track 94.2 -> 108.6 mm
- net Net-(D1-Pad1): track 13.7 -> 7.47 mm
- net GND: track 19.7 -> 15.1 mm, vias 1 -> 45
- net +5VD: track 164.2 -> 168.8 mm
- net Net-(D7-Pad2): track 0.00 -> 3.46 mm, vias 0 -> 1
- net Net-(C11-Pad1): track 47.9 -> 45.1 mm, vias 2 -> 1
- net Net-(C17-Pad1): track 40.0 -> 37.3 mm
- net Net-(J8-Pad3): track 47.4 -> 49.7 mm, vias 2 -> 1
- net Net-(J8-Pad6): track 33.1 -> 35.3 mm
- net Net-(C16-Pad1): track 32.8 -> 30.6 mm
- net Net-(J8-Pad8): track 46.1 -> 48.1 mm
- net Net-(J8-Pad7): track 50.5 -> 52.3 mm
- net Net-(J8-Pad10): track 27.4 -> 26.2 mm
- net Net-(C6-Pad1): track 12.0 -> 13.2 mm
- net Net-(C12-Pad1): track 45.1 -> 45.9 mm, vias 2 -> 0
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