File: Circuito-IO/DomPiWeb.kicad_pcb (KiCad board)
At the start: 2 copper layers, 90 x 60 mm, 63 parts, among them J1 (-)12v(+), J10 (+)S1(-), J11 (+)S2(-), J2 EXP1, J3 (+)12v(-), J4 Bx3, J5 Bx2, J6 Bx3, J7 RaspberryPi GPIO, J8 Serial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

Commit message: Correcciones de estética
Correcciones de estética
Parts:
- moved J8 5.06 mm to (153.0, 104.2), turned to -90 degrees
Connections:
- J8 pad 1: Net-(J8-Pad1) -> GND
- J8 pad 3: GND -> Net-(J8-Pad3)
- R21 pad 2: Net-(J8-Pad1) -> Net-(J8-Pad3)
Routing:
- net Net-(J8-Pad3): track 0.00 -> 15.4 mm
- net Net-(J8-Pad1): track 15.4 -> 0.00 mm
- added copper zone on F.Cu, net (none)
Other:
- board text added: "Dom32PI - Módulo de expansión"
- board text added: "Entrada"
- board text added: "Estado"
- board text added: "Fusible 12v"
- board text added: "Fusible S1 y S2"
- board text added: "G"
- board text added: "HECHO EN ARGENTINA"
- board text added: "Info"
- board text added: "Rx"
- board text added: "Salida"
- board text added: "Tx"
