File: Circuito-IO/DomPiWeb.kicad_sch (KiCad schematic)
At the start: 74 parts, among them J13 Bx2, J14 Bx2, J3 Bx3, J5 Bx2, J7 Bx3

Commit message: Placa para central con relee y sin modem
Placa para central con relee y sin modem
Parts:
- removed J2: (no value), symbol Connector_Generic:Conn_01x02
- removed J3, J7: Bx3, TerminalBlock_Phoenix:TerminalBlock_Phoenix_PT-1,5-3-5.0-H_1x03_P5.00mm_Horizontal, symbol Connector:Screw_Terminal_01x03
- removed J5: Bx2, TerminalBlock_Phoenix:TerminalBlock_Phoenix_PT-1,5-2-5.0-H_1x02_P5.00mm_Horizontal, symbol Connector:Screw_Terminal_01x02
- added J2: (no value), TerminalBlock_Phoenix:TerminalBlock_Phoenix_PT-1,5-2-5.0-H_1x02_P5.00mm_Horizontal, symbol Connector:Screw_Terminal_01x02
- added J3: (no value), symbol Connector_Generic:Conn_01x03
- added J5: (no value), symbol Connector_Generic:Conn_01x05
- C10, C11, C12, C13, C14, C15, C16, C17, C18, C4, C6, C8, C9: value (none) -> 100nf; footprint (none) -> Capacitor_SMD:C_0805_2012Metric_Pad1.18x1.45mm_HandSolder
- C19, C5: value (none) -> 470uf; footprint (none) -> Capacitor_Tantalum_SMD:CP_EIA-7343-43_Kemet-X_Pad2.25x2.55mm_HandSolder
- D1, D2: value (none) -> LL4148; footprint (none) -> Diode_SMD:D_MiniMELF
- D10: value (none) -> Led SMD; footprint (none) -> LED_SMD:LED_1206_3216Metric_Pad1.42x1.75mm_HandSolder
- D3: value (none) -> M7; footprint (none) -> Diode_SMD:D_SOD-128
- D5: value (none) -> PMEG4050EP; footprint (none) -> Diode_SMD:D_SOD-128
- J1: value (none) -> Entrada 12v; footprint (none) -> TerminalBlock_Phoenix:TerminalBlock_Phoenix_PT-1,5-2-5.0-H_1x02_P5.00mm_Horizontal
- J10, J12: value (none) -> Bx3; footprint (none) -> TerminalBlock_Phoenix:TerminalBlock_Phoenix_PT-1,5-3-5.0-H_1x03_P5.00mm_Horizontal
- J11, J9: value (none) -> Bx2; footprint (none) -> TerminalBlock_Phoenix:TerminalBlock_Phoenix_PT-1,5-2-5.0-H_1x02_P5.00mm_Horizontal
- J4: value (none) -> Salida 5v Controlada; footprint (none) -> TerminalBlock_Phoenix:TerminalBlock_Phoenix_PT-1,5-2-5.0-H_1x02_P5.00mm_Horizontal
- J6: value (none) -> RaspberryPi GPIO; footprint (none) -> Connector_PinSocket_2.54mm:PinSocket_2x20_P2.54mm_Vertical
- J8: value (none) -> EXP1; footprint (none) -> Connector_PinHeader_2.54mm:PinHeader_2x05_P2.54mm_Vertical
- K1, K2: value (none) -> FINDER-36.11; footprint (none) -> Relay_THT:Relay_SPDT_Finder_36.11
- L1: value (none) -> 47uH - SRR1210-470M; footprint (none) -> Inductor_SMD:L_Bourns_SRR1210A
- Q2: value (none) -> DMG2305UXQ6; footprint (none) -> Package_TO_SOT_SMD:SOT-23
- Q3, Q4, Q5: value (none) -> BC848; footprint (none) -> Package_TO_SOT_SMD:SOT-23
- R1, R4: value (none) -> 22R
- R13, R14: value (none) -> 22R; footprint (none) -> Resistor_SMD:R_0805_2012Metric_Pad1.20x1.40mm_HandSolder
- R16, R17, R43, R44: value (none) -> 10K; footprint (none) -> Resistor_SMD:R_0805_2012Metric_Pad1.20x1.40mm_HandSolder
- R19, R2, R22, R23, R24, R25, R26, R27, R30, R31, R32, R33, R34, R35, R36, R37, R38, R39, R40, R41, R42, R8: value (none) -> 1K; footprint (none) -> Resistor_SMD:R_0805_2012Metric_Pad1.20x1.40mm_HandSolder
- R3: value (none) -> 3K3; footprint (none) -> Resistor_SMD:R_0805_2012Metric_Pad1.20x1.40mm_HandSolder
- R9: footprint (none) -> Resistor_SMD:R_0805_2012Metric_Pad1.20x1.40mm_HandSolder
- U1: value (none) -> LM2596S-ADJ; footprint (none) -> Package_TO_SOT_SMD:TO-263-5_TabPin3
Connections:
- net +5VD: now also J2.1 (Pin_1), J5.1 (Pin_1)
- net GND: now also J2.2 (Pin_2), J3.3 (Pin_3), J5.5 (Pin_5)
- net at R9.2: now also J5.4 (Pin_4)
- net at R13.2: now also J3.1 (Pin_1)
- net at R14.2: now also J3.2 (Pin_2)
- net at R1.2: now also J5.2 (Pin_2)
- net at R4.2: now also J5.3 (Pin_3)

Commit message: Update
Update
Parts:
- J13, J14: value Bx2 -> (none); footprint TerminalBlock_Phoenix:TerminalBlock_Phoenix_PT-1,5-2-5.0-H_1x02_P5.00mm_Horizontal -> (none)
- J2: value (none) -> Salida 5v
- J3: value (none) -> Serial; footprint (none) -> Connector_PinHeader_2.54mm:PinHeader_1x03_P2.54mm_Vertical
- J5: value (none) -> EXP2; footprint (none) -> Connector_PinHeader_2.54mm:PinHeader_1x05_P2.54mm_Vertical
- R9: value (none) -> 22R
Connections:
- net at J6.19 (MOSI0/GPIO10): now also R1.1; no longer R4.1
- net at J6.21 (MISO0/GPIO9): now also R42.1; no longer R1.1
- net at J6.32 (PWM0/GPIO12): now also R4.1; no longer R9.1
- net at J6.33 (PWM1/GPIO13): now also R9.1; no longer R42.1
Changed lines of the file:
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@@
-    (stroke (width 0) (type default) (color 0 0 0 0))
-  )
-  (wire (pts (xy 135.89 128.27) (xy 138.43 128.27))
     (stroke (width 0) (type default) (color 0 0 0 0))
   )
@@
     (stroke (width 0) (type default) (color 0 0 0 0))
   )
-  (wire (pts (xy 135.89 125.73) (xy 214.63 125.73))
-    (stroke (width 0) (type default) (color 0 0 0 0))
-  )
   (wire (pts (xy 149.86 187.96) (xy 154.94 187.96))
     (stroke (width 0) (type default) (color 0 0 0 0))
@@
     (stroke (width 0) (type default) (color 0 0 0 0))
   )
+  (wire (pts (xy 135.89 118.11) (xy 212.09 118.11))
+    (stroke (width 0) (type default) (color 0 0 0 0))
+  )
   (wire (pts (xy 24.13 80.01) (xy 19.05 80.01))
     (stroke (width 0) (type default) (color 0 0 0 0))
@@
     (stroke (width 0) (type default) (color 0 0 0 0))
   )
+  (wire (pts (xy 135.89 125.73) (xy 213.36 125.73))
+    (stroke (width 0) (type default) (color 0 0 0 0))
+  )
   (wire (pts (xy 36.83 73.66) (xy 40.64 73.66))
     (stroke (width 0) (type default) (color 0 0 0 0))
   )
-  (wire (pts (xy 138.43 128.27) (xy 138.43 77.47))
-    (stroke (width 0) (type default) (color 0 0 0 0))
-  )
   (wire (pts (xy 212.09 82.55) (xy 219.71 82.55))
     (stroke (width 0) (type default) (color 0 0 0 0))
@@
     (stroke (width 0) (type default) (color 0 0 0 0))
   )
+  (wire (pts (xy 138.43 115.57) (xy 138.43 77.47))
+    (stroke (width 0) (type default) (color 0 0 0 0))
+  )
   (wire (pts (xy 34.29 146.05) (xy 33.02 146.05))
     (stroke (width 0) (type default) (color 0 0 0 0))
@@
     (stroke (width 0) (type default) (color 0 0 0 0))
   )
-  (wire (pts (xy 135.89 118.11) (xy 213.36 118.11))
-    (stroke (width 0) (type default) (color 0 0 0 0))
-  )
   (wire (pts (xy 205.74 50.8) (xy 205.74 57.15))
     (stroke (width 0) (type default) (color 0 0 0 0))
@@
     (stroke (width 0) (type default) (color 0 0 0 0))
   )
-  (wire (pts (xy 212.09 115.57) (xy 212.09 82.55))
+  (wire (pts (xy 212.09 82.55) (xy 212.09 118.11))
     (stroke (width 0) (type default) (color 0 0 0 0))
   )
@@
     (stroke (width 0) (type default) (color 0 0 0 0))
   )
-  (wire (pts (xy 214.63 125.73) (xy 214.63 87.63))
+  (wire (pts (xy 214.63 87.63) (xy 214.63 128.27))
     (stroke (width 0) (type default) (color 0 0 0 0))
   )
@@
     (stroke (width 0) (type default) (color 0 0 0 0))
   )
-  (wire (pts (xy 135.89 115.57) (xy 212.09 115.57))
-    (stroke (width 0) (type default) (color 0 0 0 0))
-  )
   (wire (pts (xy 33.02 168.91) (xy 48.26 168.91))
     (stroke (width 0) (type default) (color 0 0 0 0))
@@
     (stroke (width 0) (type default) (color 0 0 0 0))
   )
-  (wire (pts (xy 213.36 118.11) (xy 213.36 85.09))
+  (wire (pts (xy 213.36 85.09) (xy 213.36 125.73))
     (stroke (width 0) (type default) (color 0 0 0 0))
   )
@@
     (stroke (width 0) (type default) (color 0 0 0 0))
   )
+  (wire (pts (xy 135.89 115.57) (xy 138.43 115.57))
+    (stroke (width 0) (type default) (color 0 0 0 0))
+  )
   (wire (pts (xy 214.63 71.12) (xy 214.63 68.58))
     (stroke (width 0) (type default) (color 0 0 0 0))
@@
   )
   (wire (pts (xy 144.78 154.94) (xy 144.78 95.25))
+    (stroke (width 0) (type default) (color 0 0 0 0))
+  )
+  (wire (pts (xy 135.89 128.27) (xy 214.63 128.27))
     (stroke (width 0) (type default) (color 0 0 0 0))
   )
@@
     (in_bom yes) (on_board yes)
     (property "Reference" "R9" (id 0) (at 238.76 80.01 90))
-    (property "Value" "" (id 1) (at 238.76 87.63 90))
+    (property "Value" "22R" (id 1) (at 238.76 87.63 90))
     (property "Footprint" "Resistor_SMD:R_0805_2012Metric_Pad1.20x1.40mm_HandSolder" (id 2) (at 238.76 89.408 90)
       (effects (font (size 1.27 1.27)) hide)
@@
   (symbol (lib_id "Connector:Screw_Terminal_01x02") (at 254 38.1 0) (mirror x) (unit 1)
     (in_bom yes) (on_board yes)
-    (property "Reference" "J13" (id 0) (at 256.54 35.56 90)
-      (effects (font (size 1.27 1.27)) (justify left))
-    )
-    (property "Value" "Bx2" (id 1) (at 259.08 35.56 90)
-      (effects (font (size 1.27 1.27)) (justify left) hide)
-    )
-    (property "Footprint" "TerminalBlock_Phoenix:TerminalBlock_Phoenix_PT-1,5-2-5.0-H_1x02_P5.00mm_Horizontal" (id 2) (at 254 38.1 0)
+    (property "Reference" "J13" (id 0) (at 256.54 35.56 0)
+      (effects (font (size 1.27 1.27)) (justify left))
+    )
+    (property "Value" "" (id 1) (at 256.54 38.1 0)
+      (effects (font (size 1.27 1.27)) (justify left))
+    )
+    (property "Footprint" "" (id 2) (at 254 38.1 0)
       (effects (font (size 1.27 1.27)) hide)
     )
@@
       (effects (font (size 1.27 1.27)) (justify left))
     )
-    (property "Value" "" (id 1) (at 255.27 86.3599 0)
-      (effects (font (size 1.27 1.27)) (justify left))
-    )
-    (property "Footprint" "" (id 2) (at 252.73 85.09 0)
+    (property "Value" "EXP2" (id 1) (at 255.27 86.3599 0)
+      (effects (font (size 1.27 1.27)) (justify left))
+    )
+    (property "Footprint" "Connector_PinHeader_2.54mm:PinHeader_1x05_P2.54mm_Vertical" (id 2) (at 252.73 85.09 0)
       (effects (font (size 1.27 1.27)) hide)
     )
@@
   (symbol (lib_id "Connector:Screw_Terminal_01x02") (at 254 62.23 0) (mirror x) (unit 1)
     (in_bom yes) (on_board yes)
-    (property "Reference" "J14" (id 0) (at 256.54 59.69 90)
-      (effects (font (size 1.27 1.27)) (justify left))
-    )
-    (property "Value" "Bx2" (id 1) (at 259.08 59.69 90)
-      (effects (font (size 1.27 1.27)) (justify left) hide)
-    )
-    (property "Footprint" "TerminalBlock_Phoenix:TerminalBlock_Phoenix_PT-1,5-2-5.0-H_1x02_P5.00mm_Horizontal" (id 2) (at 254 62.23 0)
+    (property "Reference" "J14" (id 0) (at 256.54 59.69 0)
+      (effects (font (size 1.27 1.27)) (justify left))
+    )
+    (property "Value" "" (id 1) (at 256.54 62.23 0)
+      (effects (font (size 1.27 1.27)) (justify left))
+    )
+    (property "Footprint" "" (id 2) (at 254 62.23 0)
       (effects (font (size 1.27 1.27)) hide)
     )
@@
       (effects (font (size 1.27 1.27)) (justify left))
     )
-    (property "Value" "" (id 1) (at 119.38 63.4999 0)
-      (effects (font (size 1.27 1.27)) (justify left))
-    )
-    (property "Footprint" "" (id 2) (at 116.84 62.23 0)
+    (property "Value" "Serial" (id 1) (at 119.38 63.4999 0)
+      (effects (font (size 1.27 1.27)) (justify left))
+    )
+    (property "Footprint" "Connector_PinHeader_2.54mm:PinHeader_1x03_P2.54mm_Vertical" (id 2) (at 116.84 62.23 0)
       (effects (font (size 1.27 1.27)) hide)
     )
@@
       (effects (font (size 1.27 1.27)) (justify left))
     )
-    (property "Value" "" (id 1) (at 135.89 38.1 0)
+    (property "Value" "Salida 5v" (id 1) (at 135.89 38.1 0)
       (effects (font (size 1.27 1.27)) (justify left))
     )
@@
     )
     (path "/9104b1fe-3da9-48b2-98b4-0efb1e589f26"
-      (reference "J13") (unit 1) (value "Bx2") (footprint "TerminalBlock_Phoenix:TerminalBlock_Phoenix_PT-1,5-2-5.0-H_1x02_P5.00mm_Horizontal")
+      (reference "J13") (unit 1) (value "Salida 1") (footprint "TerminalBlock_Phoenix:TerminalBlock_Phoenix_PT-1,5-2-5.0-H_1x02_P5.00mm_Horizontal")
     )
     (path "/c181ea99-05de-49cb-8108-1619594dd4a3"
-      (reference "J14") (unit 1) (value "Bx2") (footprint "TerminalBlock_Phoenix:TerminalBlock_Phoenix_PT-1,5-2-5.0-H_1x02_P5.00mm_Horizontal")
+      (reference "J14") (unit 1) (value "Salida 2") (footprint "TerminalBlock_Phoenix:TerminalBlock_Phoenix_PT-1,5-2-5.0-H_1x02_P5.00mm_Horizontal")
     )
     (path "/60687573-08eb-47ec-9824-f6aa684b9a32"

Commit message: Nueva placa
Nueva placa
Parts:
- removed C6: 100nf, Capacitor_SMD:C_0805_2012Metric_Pad1.18x1.45mm_HandSolder, symbol Device:C
- removed J4: Salida 5v Controlada, TerminalBlock_Phoenix:TerminalBlock_Phoenix_PT-1,5-2-5.0-H_1x02_P5.00mm_Horizontal, symbol Connector:Screw_Terminal_01x02
- removed J5: EXP2, Connector_PinHeader_2.54mm:PinHeader_1x05_P2.54mm_Vertical, symbol Connector_Generic:Conn_01x05
- removed Q2: DMG2305UXQ6, Package_TO_SOT_SMD:SOT-23, symbol Device:Q_PMOS_GSD
- removed Q3: BC848, Package_TO_SOT_SMD:SOT-23, symbol Device:Q_NPN_BEC
- removed R1, R4, R9: 22R, Resistor_SMD:R_0805_2012Metric_Pad1.20x1.40mm_HandSolder, symbol Device:R
- removed R16, R17, R43, R44: 10K, Resistor_SMD:R_0805_2012Metric_Pad1.20x1.40mm_HandSolder, symbol Device:R
- removed R19, R41: 1K, Resistor_SMD:R_0805_2012Metric_Pad1.20x1.40mm_HandSolder, symbol Device:R
- added D3: Led SMD, LED_SMD:LED_1206_3216Metric_Pad1.42x1.75mm_HandSolder, symbol Device:LED
- added F1, F2: Fuse, Fuse:Fuseholder_Cylinder-5x20mm_Schurter_0031_8201_Horizontal_Open, symbol Device:Fuse
- added R2: 1K, Resistor_SMD:R_0805_2012Metric_Pad1.20x1.40mm_HandSolder, symbol Device:R
- J10: renamed from J13; value (none) -> Salida 1; footprint (none) -> TerminalBlock_Phoenix:TerminalBlock_Phoenix_PT-1,5-2-5.0-H_1x02_P5.00mm_Horizontal
- J11: renamed from J14; value (none) -> Salida 2; footprint (none) -> TerminalBlock_Phoenix:TerminalBlock_Phoenix_PT-1,5-2-5.0-H_1x02_P5.00mm_Horizontal
- R23: renamed from R8; value 1K -> 10K
- R24: renamed from R42; value 1K -> 10K
- renumbered C8 to C1, C13 to C10, C14 to C11, C15 to C12, C16 to C13, C17 to C14, C18 to C2, C9 to C3, C19 to C4, C10 to C5, C4 to C6, C11 to C7, C12 to C8, C5 to C9, D3 to D1, D10 to D2, D5 to D4, D1 to D5, D2 to D6, J8 to J2, J9 to J3, J10 to J4, J11 to J5, J12 to J6, J6 to J7, J3 to J8, J2 to J9, Q5 to Q1, Q4 to Q2, R32 to R1, R31 to R10, R33 to R11, R34 to R12, R35 to R13, R36 to R14, R37 to R15, R38 to R16, R39 to R17, R2 to R18, R40 to R19, R3 to R20, R13 to R21, R14 to R22, R22 to R3, R23 to R4, R24 to R5, R25 to R6, R26 to R7, R27 to R8, R30 to R9
Connections:
- net GND: now also J10.1 (Pin_1), J11.1 (Pin_1), D3.1 (K)
- net at J7.12 (GPIO18/PWM0): no longer R5.2
- net at J7.13 (GPIO27): now also R3.2
- net at J7.15 (GPIO22): now also R6.2; no longer R9.2
- net at J7.16 (GPIO23): now also R1.1; no longer R10.2
- net at J7.18 (GPIO24): now also R2.1
- net at J7.19 (MOSI0/GPIO10): now also R5.2
- net at J7.21 (MISO0/GPIO9): now also R8.2; no longer R24.1
- net at J7.22 (GPIO25): now also C5.1, R19.2
- net at J7.23 (SCLK0/GPIO11): now also R7.2; no longer R23.1
- net at J7.24 (~{CE0}/GPIO8): now also C7.1, R17.2; no longer R1.2
- net at C14.1, R11.2: now also J7.40 (GPIO21/SCLK1); no longer J7.27 (ID_SD/GPIO0)
- net at C13.1, R12.2: now also J7.38 (GPIO20/MOSI1); no longer J7.28 (ID_SC/GPIO1)
- net at C8.1, R16.2: now also J7.26 (~{CE1}/GPIO7); no longer J7.29 (GCLK1/GPIO5)
- net at C12.1, R13.2: now also J7.36 (GPIO16); no longer J7.3 (SDA/GPIO2)
- net at J7.32 (PWM0/GPIO12): now also C11.1, R14.2
- net at J7.35 (GPIO19/MISO1): no longer R6.2
- net at C10.1, R15.2: now also J7.28 (ID_SC/GPIO1); no longer J7.7 (GCLK0/GPIO4)
- net at D2.2 (A): now also R1.2; no longer R1.1
- net at C2.1, C4.1, D1.1 (K)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: now also F1.1; no longer D5.1 (K), D6.1 (K), K1.A1, K2.A1
- net at D1.2 (A), J1.1 (Pin_1): now also F2.1
- net at K1.11: now also J10.2 (Pin_2); no longer J10.1 (Pin_1)
- net at K1.14: now also D5.1 (K), D6.1 (K), K1.A1, K2.14, K2.A1, F2.2; no longer J10.2 (Pin_2)
- net at K2.11: now also J11.2 (Pin_2); no longer J11.1 (Pin_1)
- net +5VD: no longer names the net of C1.1, C6.1, C9.1, J2.1 (Pin_1), J9.1 (Pin_1), L1.2, R20.1
- net +5VD: no longer C3.1, J3.1 (Pin_1)
- new net: J7.27 (ID_SD/GPIO0), R10.2
- new net: J7.29 (GCLK1/GPIO5), R9.2
- new net: J7.5 (SCL/GPIO3), R23.1
- new net: J7.7 (GCLK0/GPIO4), R24.1
- new net: C3.1, F1.2, J3.1 (Pin_1)
- new net: D3.2 (A), R2.2
- now unconnected: J7.31 (GCLK2/GPIO6)
Other:
- note added: "+12v"
- note removed: "+5v"
- moved on the sheet: C1, C10, C11, C12, C13, C14, C3, C5, C7, C8, D2, J3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
