File: Circuito-IO/DomPiWeb.kicad_sch (KiCad schematic)
At the start: 63 parts, among them J1 Entrada 12v, J10 Salida 1, J11 Salida 2, J2 EXP1, J3 Bx2, J4 Bx3, J5 Bx2, J6 Bx3, J7 RaspberryPi GPIO, J8 Serial, J9 Salida 5v, K1 FINDER-36.11, K2 FINDER-36.11, Q1 BC848, Q2 BC848, U1 LM2596S-ADJ

Commit message: Update DomPiWeb.kicad_sch
Parts:
- C4: value 470uf -> (none); footprint Capacitor_Tantalum_SMD:CP_EIA-7343-43_Kemet-X_Pad2.25x2.55mm_HandSolder -> (none)
Connections:
- net at J7.2 (5V): now also C1.1, C6.1, C9.1, J2.1 (Pin_1), J7.4 (5V), J9.1 (Pin_1), L1.2, R20.1
Other:
- moved on the sheet: J8, R21, R22
Changed lines of the file:
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@@
   (junction (at 85.09 36.83) (diameter 0) (color 0 0 0 0)
   )
+  (junction (at 121.92 36.83) (diameter 0) (color 0 0 0 0)
+  )
   (junction (at 50.8 36.83) (diameter 0) (color 0 0 0 0)
   )
@@
   (junction (at 110.49 187.96) (diameter 0) (color 0 0 0 0)
   )
+  (junction (at 113.03 64.77) (diameter 0) (color 0 0 0 0)
+  )
   (junction (at 227.33 16.51) (diameter 0) (color 0 0 0 0)
   )
@@
     (stroke (width 0) (type default) (color 0 0 0 0))
   )
+  (wire (pts (xy 110.49 64.77) (xy 113.03 64.77))
+    (stroke (width 0) (type default) (color 0 0 0 0))
+  )
   (wire (pts (xy 110.49 185.42) (xy 110.49 187.96))
     (stroke (width 0) (type default) (color 0 0 0 0))
@@
     (stroke (width 0) (type default) (color 0 0 0 0))
   )
+  (wire (pts (xy 113.03 64.77) (xy 113.03 74.93))
+    (stroke (width 0) (type default) (color 0 0 0 0))
+  )
   (wire (pts (xy 140.97 162.56) (xy 105.41 162.56))
     (stroke (width 0) (type default) (color 0 0 0 0))
@@
     (stroke (width 0) (type default) (color 0 0 0 0))
   )
+  (wire (pts (xy 110.49 74.93) (xy 110.49 64.77))
+    (stroke (width 0) (type default) (color 0 0 0 0))
+  )
   (wire (pts (xy 57.15 16.51) (xy 201.93 16.51))
     (stroke (width 0) (type default) (color 0 0 0 0))
@@
     (stroke (width 0) (type default) (color 0 0 0 0))
   )
-  (wire (pts (xy 92.71 59.69) (xy 96.52 59.69))
+  (wire (pts (xy 92.71 59.69) (xy 93.98 59.69))
     (stroke (width 0) (type default) (color 0 0 0 0))
   )
@@
     (stroke (width 0) (type default) (color 0 0 0 0))
   )
-  (wire (pts (xy 93.98 62.23) (xy 101.6 62.23))
+  (wire (pts (xy 93.98 62.23) (xy 95.25 62.23))
     (stroke (width 0) (type default) (color 0 0 0 0))
   )
@@
     (stroke (width 0) (type default) (color 0 0 0 0))
   )
+  (wire (pts (xy 113.03 64.77) (xy 121.92 64.77))
+    (stroke (width 0) (type default) (color 0 0 0 0))
+  )
   (wire (pts (xy 135.89 177.8) (xy 135.89 147.32))
     (stroke (width 0) (type default) (color 0 0 0 0))
@@
     (stroke (width 0) (type default) (color 0 0 0 0))
   )
-  (wire (pts (xy 111.76 64.77) (xy 109.22 64.77))
-    (stroke (width 0) (type default) (color 0 0 0 0))
-  )
   (wire (pts (xy 24.13 146.05) (xy 24.13 148.59))
     (stroke (width 0) (type default) (color 0 0 0 0))
@@
     (stroke (width 0) (type default) (color 0 0 0 0))
   )
-  (wire (pts (xy 104.14 59.69) (xy 111.76 59.69))
+  (wire (pts (xy 101.6 59.69) (xy 102.87 59.69))
     (stroke (width 0) (type default) (color 0 0 0 0))
   )
@@
     (stroke (width 0) (type default) (color 0 0 0 0))
   )
-  (wire (pts (xy 109.22 62.23) (xy 111.76 62.23))
-    (stroke (width 0) (type default) (color 0 0 0 0))
-  )
   (wire (pts (xy 95.25 105.41) (xy 91.44 105.41))
     (stroke (width 0) (type default) (color 0 0 0 0))
@@
     (stroke (width 0) (type default) (color 0 0 0 0))
   )
+  (wire (pts (xy 121.92 64.77) (xy 121.92 36.83))
+    (stroke (width 0) (type default) (color 0 0 0 0))
+  )
   (wire (pts (xy 135.89 187.96) (xy 135.89 194.31))
     (stroke (width 0) (type default) (color 0 0 0 0))
@@
     (stroke (width 0) (type default) (color 0 0 0 0))
   )
-  (wire (pts (xy 109.22 64.77) (xy 109.22 67.31))
+  (wire (pts (xy 102.87 64.77) (xy 102.87 66.04))
     (stroke (width 0) (type default) (color 0 0 0 0))
   )
@@
     (stroke (width 0) (type default) (color 0 0 0 0))
   )
-  (wire (pts (xy 128.27 36.83) (xy 113.03 36.83))
+  (wire (pts (xy 128.27 36.83) (xy 121.92 36.83))
     (stroke (width 0) (type default) (color 0 0 0 0))
   )
@@
   )
   (wire (pts (xy 115.57 177.8) (xy 115.57 157.48))
+    (stroke (width 0) (type default) (color 0 0 0 0))
+  )
+  (wire (pts (xy 121.92 36.83) (xy 113.03 36.83))
     (stroke (width 0) (type default) (color 0 0 0 0))
   )
@@
     (pin "2")
   )
-  (symbol (lib_id "Device:R") (at 100.33 59.69 90) (unit 1)
-    (in_bom yes) (on_board yes)
-    (property "Reference" "R21" (id 0) (at 100.33 57.15 90))
-    (property "Value" "22R" (id 1) (at 100.33 59.69 90))
-    (property "Footprint" "Resistor_SMD:R_0805_2012Metric_Pad1.20x1.40mm_HandSolder" (id 2) (at 100.33 61.468 90)
-      (effects (font (size 1.27 1.27)) hide)
-    )
-    (property "Datasheet" "~" (id 3) (at 100.33 59.69 0)
-      (effects (font (size 1.27 1.27)) hide)
-    )
-    (pin "1")
-    (pin "2")
-  )
-  (symbol (lib_id "Device:R") (at 105.41 62.23 90) (unit 1)
-    (in_bom yes) (on_board yes)
-    (property "Reference" "R22" (id 0) (at 105.41 64.77 90))
-    (property "Value" "22R" (id 1) (at 105.41 62.23 90))
-    (property "Footprint" "Resistor_SMD:R_0805_2012Metric_Pad1.20x1.40mm_HandSolder" (id 2) (at 105.41 64.008 90)
-      (effects (font (size 1.27 1.27)) hide)
-    )
-    (property "Datasheet" "~" (id 3) (at 105.41 62.23 0)
+  (symbol (lib_id "Device:R") (at 97.79 59.69 90) (unit 1)
+    (in_bom yes) (on_board yes)
+    (property "Reference" "R21" (id 0) (at 97.79 57.15 90))
+    (property "Value" "22R" (id 1) (at 97.79 59.69 90))
+    (property "Footprint" "Resistor_SMD:R_0805_2012Metric_Pad1.20x1.40mm_HandSolder" (id 2) (at 97.79 61.468 90)
+      (effects (font (size 1.27 1.27)) hide)
+    )
+    (property "Datasheet" "~" (id 3) (at 97.79 59.69 0)
+      (effects (font (size 1.27 1.27)) hide)
+    )
+    (pin "1")
+    (pin "2")
+  )
+  (symbol (lib_id "Device:R") (at 99.06 62.23 90) (unit 1)
+    (in_bom yes) (on_board yes)
+    (property "Reference" "R22" (id 0) (at 99.06 64.77 90))
+    (property "Value" "22R" (id 1) (at 99.06 62.23 90))
+    (property "Footprint" "Resistor_SMD:R_0805_2012Metric_Pad1.20x1.40mm_HandSolder" (id 2) (at 99.06 64.008 90)
+      (effects (font (size 1.27 1.27)) hide)
+    )
+    (property "Datasheet" "~" (id 3) (at 99.06 62.23 0)
       (effects (font (size 1.27 1.27)) hide)
     )
@@
       (effects (font (size 1.27 1.27)) (justify left))
     )
-    (property "Value" "470uf" (id 1) (at 51.2572 51.943 0)
-      (effects (font (size 1.27 1.27)) (justify left))
-    )
-    (property "Footprint" "Capacitor_Tantalum_SMD:CP_EIA-7343-43_Kemet-X_Pad2.25x2.55mm_HandSolder" (id 2) (at 49.2252 54.61 0)
+    (property "Value" "" (id 1) (at 51.2572 51.943 0)
+      (effects (font (size 1.27 1.27)) (justify left))
+    )
+    (property "Footprint" "" (id 2) (at 49.2252 54.61 0)
       (effects (font (size 1.27 1.27)) hide)
     )
@@
     (pin "1")
   )
-  (symbol (lib_id "power:GND") (at 109.22 67.31 0) (unit 1)
-    (in_bom yes) (on_board yes)
-    (property "Reference" "#PWR011" (id 0) (at 109.22 73.66 0)
-      (effects (font (size 1.27 1.27)) hide)
-    )
-    (property "Value" "GND" (id 1) (at 109.347 71.7042 0)
-      (effects (font (size 1.27 1.27)) hide)
-    )
-    (property "Footprint" "" (id 2) (at 109.22 67.31 0)
-      (effects (font (size 1.27 1.27)) hide)
-    )
-    (property "Datasheet" "" (id 3) (at 109.22 67.31 0)
+  (symbol (lib_id "power:GND") (at 102.87 66.04 0) (unit 1)
+    (in_bom yes) (on_board yes)
+    (property "Reference" "#PWR011" (id 0) (at 102.87 72.39 0)
+      (effects (font (size 1.27 1.27)) hide)
+    )
+    (property "Value" "GND" (id 1) (at 102.997 70.4342 0)
+      (effects (font (size 1.27 1.27)) hide)
+    )
+    (property "Footprint" "" (id 2) (at 102.87 66.04 0)
+      (effects (font (size 1.27 1.27)) hide)
+    )
+    (property "Datasheet" "" (id 3) (at 102.87 66.04 0)
       (effects (font (size 1.27 1.27)) hide)
     )
@@
     (pin "2")
   )
-  (symbol (lib_id "Connector_Generic:Conn_01x03") (at 116.84 62.23 0) (unit 1)
+  (symbol (lib_id "Connector_Generic:Conn_01x03") (at 107.95 62.23 0) (unit 1)
     (in_bom yes) (on_board yes) (fields_autoplaced)
-    (property "Reference" "J8" (id 0) (at 119.38 60.9599 0)
-      (effects (font (size 1.27 1.27)) (justify left))
-    )
-    (property "Value" "Serial" (id 1) (at 119.38 63.4999 0)
-      (effects (font (size 1.27 1.27)) (justify left))
-    )
-    (property "Footprint" "Connector_PinHeader_2.54mm:PinHeader_1x03_P2.54mm_Vertical" (id 2) (at 116.84 62.23 0)
-      (effects (font (size 1.27 1.27)) hide)
-    )
-    (property "Datasheet" "~" (id 3) (at 116.84 62.23 0)
+    (property "Reference" "J8" (id 0) (at 110.49 60.9599 0)
+      (effects (font (size 1.27 1.27)) (justify left))
+    )
+    (property "Value" "Serial" (id 1) (at 110.49 63.4999 0)
+      (effects (font (size 1.27 1.27)) (justify left))
+    )
+    (property "Footprint" "Connector_PinHeader_2.54mm:PinHeader_1x03_P2.54mm_Vertical" (id 2) (at 107.95 62.23 0)
+      (effects (font (size 1.27 1.27)) hide)
+    )
+    (property "Datasheet" "~" (id 3) (at 107.95 62.23 0)
       (effects (font (size 1.27 1.27)) hide)
     )
@@
     )
     (path "/00000000-0000-0000-0000-00006269f193"
-      (reference "C4") (unit 1) (value "470uf") (footprint "Capacitor_Tantalum_SMD:CP_EIA-7343-43_Kemet-X_Pad2.25x2.55mm_HandSolder")
+      (reference "C4") (unit 1) (value "10uf") (footprint "Capacitor_Tantalum_SMD:CP_EIA-7343-43_Kemet-X_Pad2.25x2.55mm_HandSolder")
     )
     (path "/00000000-0000-0000-0000-000060f609c6"

Commit message: PCB completo
PCB completo. Con cambios en leyendas y en el esquema para simplificar el PCB
Parts:
- C4: value (none) -> 10uf; footprint (none) -> Capacitor_Tantalum_SMD:CP_EIA-7343-43_Kemet-X_Pad2.25x2.55mm_HandSolder
- J1: value Entrada 12v -> (none)
- J10: value Salida 1 -> (none)
- J11: value Salida 2 -> (none)
- J3: value Bx2 -> (none); footprint TerminalBlock_Phoenix:TerminalBlock_Phoenix_PT-1,5-2-5.0-H_1x02_P5.00mm_Horizontal -> (none)
- J9: value Salida 5v -> (none); footprint TerminalBlock_Phoenix:TerminalBlock_Phoenix_PT-1,5-2-5.0-H_1x02_P5.00mm_Horizontal -> (none)
Connections:
- net GND: now also J10.2 (Pin_2), J11.2 (Pin_2); no longer J10.1 (Pin_1), J11.1 (Pin_1)
- net at K1.11: now also J10.1 (Pin_1); no longer J10.2 (Pin_2)
- net at K2.11: now also J11.1 (Pin_1); no longer J11.2 (Pin_2)
Other:
- note removed: "+12v"
- note removed: "Gnd"
Changed lines of the file:
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@@
+    (stroke (width 0) (type default) (color 0 0 0 0))
+  )
+  (wire (pts (xy 246.38 38.1) (xy 248.92 38.1))
     (stroke (width 0) (type default) (color 0 0 0 0))
   )
@@
     (stroke (width 0) (type default) (color 0 0 0 0))
   )
-  (wire (pts (xy 248.92 62.23) (xy 246.38 62.23))
-    (stroke (width 0) (type default) (color 0 0 0 0))
-  )
   (wire (pts (xy 205.74 40.64) (xy 205.74 46.99))
     (stroke (width 0) (type default) (color 0 0 0 0))
@@
     (stroke (width 0) (type default) (color 0 0 0 0))
   )
-  (wire (pts (xy 248.92 38.1) (xy 246.38 38.1))
-    (stroke (width 0) (type default) (color 0 0 0 0))
-  )
   (wire (pts (xy 88.9 21.59) (xy 86.36 21.59))
     (stroke (width 0) (type default) (color 0 0 0 0))
@@
   )
   (wire (pts (xy 214.63 26.67) (xy 205.74 26.67))
+    (stroke (width 0) (type default) (color 0 0 0 0))
+  )
+  (wire (pts (xy 246.38 62.23) (xy 248.92 62.23))
     (stroke (width 0) (type default) (color 0 0 0 0))
   )
@@
     (effects (font (size 2.4892 2.4892) (thickness 0.4978) bold) (justify left bottom))
   )
-  (text "Gnd" (at 58.42 196.85 90)
-    (effects (font (size 1.27 1.27)) (justify left bottom))
-  )
   (text "IO6" (at 73.66 196.85 90)
     (effects (font (size 1.27 1.27)) (justify left bottom))
@@
   (text "IO7" (at 76.2 196.85 90)
     (effects (font (size 1.27 1.27)) (justify left bottom))
-  )
-  (text "+12v" (at 55.88 193.04 270)
-    (effects (font (size 1.27 1.27)) (justify right bottom))
   )
   (symbol (lib_id "Connector:Raspberry_Pi_2_3") (at 115.57 107.95 0) (unit 1)
@@
       (effects (font (size 1.27 1.27)) (justify left))
     )
-    (property "Value" "Bx2" (id 1) (at 58.42 195.58 90)
-      (effects (font (size 1.27 1.27)) (justify left) hide)
-    )
-    (property "Footprint" "TerminalBlock_Phoenix:TerminalBlock_Phoenix_PT-1,5-2-5.0-H_1x02_P5.00mm_Horizontal" (id 2) (at 55.88 190.5 0)
+    (property "Value" "" (id 1) (at 58.42 195.58 90)
+      (effects (font (size 1.27 1.27)) (justify left))
+    )
+    (property "Footprint" "" (id 2) (at 55.88 190.5 0)
       (effects (font (size 1.27 1.27)) hide)
     )
@@
       (effects (font (size 1.27 1.27)) (justify left))
     )
-    (property "Value" "Entrada 12v" (id 1) (at 26.67 33.02 0)
+    (property "Value" "" (id 1) (at 26.67 33.02 0)
       (effects (font (size 1.27 1.27)) (justify left))
     )
@@
       (effects (font (size 1.27 1.27)) (justify left))
     )
-    (property "Value" "" (id 1) (at 51.2572 51.943 0)
-      (effects (font (size 1.27 1.27)) (justify left))
-    )
-    (property "Footprint" "" (id 2) (at 49.2252 54.61 0)
+    (property "Value" "10uf" (id 1) (at 51.2572 51.943 0)
+      (effects (font (size 1.27 1.27)) (justify left))
+    )
+    (property "Footprint" "Capacitor_Tantalum_SMD:CP_EIA-7343-43_Kemet-X_Pad2.25x2.55mm_HandSolder" (id 2) (at 49.2252 54.61 0)
       (effects (font (size 1.27 1.27)) hide)
     )
@@
     (pin "2")
   )
-  (symbol (lib_id "Connector:Screw_Terminal_01x02") (at 254 38.1 0) (mirror x) (unit 1)
-    (in_bom yes) (on_board yes)
-    (property "Reference" "J10" (id 0) (at 256.54 35.56 0)
-      (effects (font (size 1.27 1.27)) (justify left))
-    )
-    (property "Value" "Salida 1" (id 1) (at 256.54 38.1 0)
-      (effects (font (size 1.27 1.27)) (justify left))
-    )
-    (property "Footprint" "TerminalBlock_Phoenix:TerminalBlock_Phoenix_PT-1,5-2-5.0-H_1x02_P5.00mm_Horizontal" (id 2) (at 254 38.1 0)
-      (effects (font (size 1.27 1.27)) hide)
-    )
-    (property "Datasheet" "~" (id 3) (at 254 38.1 0)
-      (effects (font (size 1.27 1.27)) hide)
-    )
-    (pin "1")
-    (pin "2")
-  )
-  (symbol (lib_id "Connector:Screw_Terminal_01x02") (at 254 62.23 0) (mirror x) (unit 1)
-    (in_bom yes) (on_board yes)
-    (property "Reference" "J11" (id 0) (at 256.54 59.69 0)
-      (effects (font (size 1.27 1.27)) (justify left))
-    )
-    (property "Value" "Salida 2" (id 1) (at 256.54 62.23 0)
-      (effects (font (size 1.27 1.27)) (justify left))
-    )
-    (property "Footprint" "TerminalBlock_Phoenix:TerminalBlock_Phoenix_PT-1,5-2-5.0-H_1x02_P5.00mm_Horizontal" (id 2) (at 254 62.23 0)
-      (effects (font (size 1.27 1.27)) hide)
-    )
-    (property "Datasheet" "~" (id 3) (at 254 62.23 0)
+  (symbol (lib_id "Connector:Screw_Terminal_01x02") (at 254 35.56 0) (unit 1)
+    (in_bom yes) (on_board yes)
+    (property "Reference" "J10" (id 0) (at 256.54 38.1 0)
+      (effects (font (size 1.27 1.27)) (justify left))
+    )
+    (property "Value" "" (id 1) (at 256.54 35.56 0)
+      (effects (font (size 1.27 1.27)) (justify left))
+    )
+    (property "Footprint" "TerminalBlock_Phoenix:TerminalBlock_Phoenix_PT-1,5-2-5.0-H_1x02_P5.00mm_Horizontal" (id 2) (at 254 35.56 0)
+      (effects (font (size 1.27 1.27)) hide)
+    )
+    (property "Datasheet" "~" (id 3) (at 254 35.56 0)
+      (effects (font (size 1.27 1.27)) hide)
+    )
+    (pin "1")
+    (pin "2")
+  )
+  (symbol (lib_id "Connector:Screw_Terminal_01x02") (at 254 59.69 0) (unit 1)
+    (in_bom yes) (on_board yes)
+    (property "Reference" "J11" (id 0) (at 256.54 62.23 0)
+      (effects (font (size 1.27 1.27)) (justify left))
+    )
+    (property "Value" "" (id 1) (at 256.54 59.69 0)
+      (effects (font (size 1.27 1.27)) (justify left))
+    )
+    (property "Footprint" "TerminalBlock_Phoenix:TerminalBlock_Phoenix_PT-1,5-2-5.0-H_1x02_P5.00mm_Horizontal" (id 2) (at 254 59.69 0)
+      (effects (font (size 1.27 1.27)) hide)
+    )
+    (property "Datasheet" "~" (id 3) (at 254 59.69 0)
       (effects (font (size 1.27 1.27)) hide)
     )
@@
       (effects (font (size 1.27 1.27)) (justify left))
     )
-    (property "Value" "Salida 5v" (id 1) (at 135.89 38.1 0)
-      (effects (font (size 1.27 1.27)) (justify left))
-    )
-    (property "Footprint" "TerminalBlock_Phoenix:TerminalBlock_Phoenix_PT-1,5-2-5.0-H_1x02_P5.00mm_Horizontal" (id 2) (at 133.35 36.83 0)
+    (property "Value" "" (id 1) (at 135.89 38.1 0)
+      (effects (font (size 1.27 1.27)) (justify left))
+    )
+    (property "Footprint" "" (id 2) (at 133.35 36.83 0)
       (effects (font (size 1.27 1.27)) hide)
     )
@@
     )
     (path "/00000000-0000-0000-0000-0000610cf2ea"
-      (reference "J1") (unit 1) (value "Entrada 12v") (footprint "TerminalBlock_Phoenix:TerminalBlock_Phoenix_PT-1,5-2-5.0-H_1x02_P5.00mm_Horizontal")
+      (reference "J1") (unit 1) (value "(-)12v(+)") (footprint "TerminalBlock_Phoenix:TerminalBlock_Phoenix_PT-1,5-2-5.0-H_1x02_P5.00mm_Horizontal")
     )
     (path "/00000000-0000-0000-0000-000060e87291"
@@
     )
     (path "/00000000-0000-0000-0000-00006095705b"
-      (reference "J3") (unit 1) (value "Bx2") (footprint "TerminalBlock_Phoenix:TerminalBlock_Phoenix_PT-1,5-2-5.0-H_1x02_P5.00mm_Horizontal")
+      (reference "J3") (unit 1) (value "(+)12v(-)") (footprint "TerminalBlock_Phoenix:TerminalBlock_Phoenix_PT-1,5-2-5.0-H_1x02_P5.00mm_Horizontal")
     )
     (path "/00000000-0000-0000-0000-000060958ac0"
@@
     )
     (path "/ed8c2c79-9a57-47de-9e2d-cc26af4b1fcc"
-      (reference "J9") (unit 1) (value "Salida 5v") (footprint "TerminalBlock_Phoenix:TerminalBlock_Phoenix_PT-1,5-2-5.0-H_1x02_P5.00mm_Horizontal")
+      (reference "J9") (unit 1) (value "(-)5v(+)") (footprint "TerminalBlock_Phoenix:TerminalBlock_Phoenix_PT-1,5-2-5.0-H_1x02_P5.00mm_Horizontal")
     )
     (path "/9104b1fe-3da9-48b2-98b4-0efb1e589f26"
-      (reference "J10") (unit 1) (value "Salida 1") (footprint "TerminalBlock_Phoenix:TerminalBlock_Phoenix_PT-1,5-2-5.0-H_1x02_P5.00mm_Horizontal")
+      (reference "J10") (unit 1) (value "(+)S1(-)") (footprint "TerminalBlock_Phoenix:TerminalBlock_Phoenix_PT-1,5-2-5.0-H_1x02_P5.00mm_Horizontal")
     )
     (path "/c181ea99-05de-49cb-8108-1619594dd4a3"
-      (reference "J11") (unit 1) (value "Salida 2") (footprint "TerminalBlock_Phoenix:TerminalBlock_Phoenix_PT-1,5-2-5.0-H_1x02_P5.00mm_Horizontal")
+      (reference "J11") (unit 1) (value "(+)S2(-)") (footprint "TerminalBlock_Phoenix:TerminalBlock_Phoenix_PT-1,5-2-5.0-H_1x02_P5.00mm_Horizontal")
     )
     (path "/60687573-08eb-47ec-9824-f6aa684b9a32"

Commit message: Correcciones de estética
Correcciones de estética
Parts:
- J1: value (none) -> (-)12v(+)
- J10: value (none) -> (+)S1(-)
- J11: value (none) -> (+)S2(-)
- J3: value (none) -> (+)12v(-); footprint (none) -> TerminalBlock_Phoenix:TerminalBlock_Phoenix_PT-1,5-2-5.0-H_1x02_P5.00mm_Horizontal
- J9: value (none) -> (-)5v(+); footprint (none) -> TerminalBlock_Phoenix:TerminalBlock_Phoenix_PT-1,5-2-5.0-H_1x02_P5.00mm_Horizontal
Connections:
- net GND: now also J8.1 (Pin_1); no longer J8.3 (Pin_3)
- net at R21.2: now also J8.3 (Pin_3); no longer J8.1 (Pin_1)
Changed lines of the file:
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@@
     (in_bom yes) (on_board yes)
     (property "Reference" "J7" (id 0) (at 99.06 74.93 0))
-    (property "Value" "RaspberryPi GPIO" (id 1) (at 124.46 71.12 0))
+    (property "Value" "RaspberryPi GPIO" (id 1) (at 130.81 74.93 0))
     (property "Footprint" "Connector_PinSocket_2.54mm:PinSocket_2x20_P2.54mm_Vertical" (id 2) (at 115.57 107.95 0)
       (effects (font (size 1.27 1.27)) hide)
@@
       (effects (font (size 1.27 1.27)) (justify left))
     )
-    (property "Value" "" (id 1) (at 58.42 195.58 90)
-      (effects (font (size 1.27 1.27)) (justify left))
-    )
-    (property "Footprint" "" (id 2) (at 55.88 190.5 0)
+    (property "Value" "(+)12v(-)" (id 1) (at 58.42 195.58 90)
+      (effects (font (size 1.27 1.27)) (justify left))
+    )
+    (property "Footprint" "TerminalBlock_Phoenix:TerminalBlock_Phoenix_PT-1,5-2-5.0-H_1x02_P5.00mm_Horizontal" (id 2) (at 55.88 190.5 0)
       (effects (font (size 1.27 1.27)) hide)
     )
@@
       (effects (font (size 1.27 1.27)) (justify left))
     )
-    (property "Value" "" (id 1) (at 26.67 33.02 0)
+    (property "Value" "(-)12v(+)" (id 1) (at 26.67 33.02 0)
       (effects (font (size 1.27 1.27)) (justify left))
     )
@@
       (effects (font (size 1.27 1.27)) (justify left))
     )
-    (property "Value" "" (id 1) (at 256.54 35.56 0)
+    (property "Value" "(+)S1(-)" (id 1) (at 256.54 35.56 0)
       (effects (font (size 1.27 1.27)) (justify left))
     )
@@
       (effects (font (size 1.27 1.27)) (justify left))
     )
-    (property "Value" "" (id 1) (at 256.54 59.69 0)
+    (property "Value" "(+)S2(-)" (id 1) (at 256.54 59.69 0)
       (effects (font (size 1.27 1.27)) (justify left))
     )
@@
     (pin "2")
   )
-  (symbol (lib_id "Connector_Generic:Conn_01x03") (at 107.95 62.23 0) (unit 1)
-    (in_bom yes) (on_board yes) (fields_autoplaced)
-    (property "Reference" "J8" (id 0) (at 110.49 60.9599 0)
-      (effects (font (size 1.27 1.27)) (justify left))
-    )
-    (property "Value" "Serial" (id 1) (at 110.49 63.4999 0)
-      (effects (font (size 1.27 1.27)) (justify left))
-    )
+  (symbol (lib_id "Connector_Generic:Conn_01x03") (at 107.95 62.23 0) (mirror x) (unit 1)
+    (in_bom yes) (on_board yes)
+    (property "Reference" "J8" (id 0) (at 111.76 58.42 0))
+    (property "Value" "Serial" (id 1) (at 113.03 60.96 0))
     (property "Footprint" "Connector_PinHeader_2.54mm:PinHeader_1x03_P2.54mm_Vertical" (id 2) (at 107.95 62.23 0)
       (effects (font (size 1.27 1.27)) hide)
@@
       (effects (font (size 1.27 1.27)) (justify left))
     )
-    (property "Value" "" (id 1) (at 135.89 38.1 0)
-      (effects (font (size 1.27 1.27)) (justify left))
-    )
-    (property "Footprint" "" (id 2) (at 133.35 36.83 0)
-      (effects (font (size 1.27 1.27)) hide)
-    )
+    (property "Value" "(-)5v(+)" (id 1) (at 135.89 38.1 0)
+      (effects (font (size 1.27 1.27)) (justify left))
+    )
+    (property "Footprint" "TerminalBlock_Phoenix:TerminalBlock_Phoenix_PT-1,5-2-5.0-H_1x02_P5.00mm_Horizontal" (id 2) (at 133.35 36.83 0)
+      (effects (font (size 1.27 1.27)) hide)
+    )
